File: hw/numitron clock-rotated-numitrons_smd.kicad_pcb (KiCad board)
At the start: 2 copper layers, 120 x 50.2 mm, 25 parts, among them J1 AVR-ISP-6, J3 5v in, J4 UART, SW2 Set M, SW3 Set H, U1 TPIC6595, U2 TPIC6595, U3 TPIC6595, U4 TPIC6595, U5 ATmega8L-8A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

Commit message: version of pcb with more smd components
Parts:
- added REF**: MountingHole_4mm, MountingHole:MountingHole_4mm, F.Cu at (158.5, 122.5)
Routing:
- net GNDREF: track 0.00 -> 411.8 mm, vias 0 -> 2
- net VCC: track 0.00 -> 302.8 mm, vias 0 -> 2
- net SRCLR: track 0.00 -> 121.5 mm, vias 0 -> 4
- net RCLK: track 0.00 -> 120.2 mm, vias 0 -> 3
- net SRCK: track 0.00 -> 114.5 mm, vias 0 -> 2
- net RXD: track 0.00 -> 78.8 mm, vias 0 -> 1
- net Net-(SW2-Pad1): track 0.00 -> 75.8 mm
- net G3: track 0.00 -> 69.8 mm, vias 0 -> 2
- net Net-(SW3-Pad1): track 0.00 -> 64.7 mm
- net G4: track 0.00 -> 63.4 mm
- net TXD: track 0.00 -> 62.4 mm, vias 0 -> 1
- net SD3: track 0.00 -> 58.7 mm, vias 0 -> 2
- net RST: track 0.00 -> 56.3 mm, vias 0 -> 1
- net SD4: track 0.00 -> 55.0 mm
- net Net-(D1-Pad2): track 0.00 -> 38.1 mm
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
Commit message: updates
Parts:
- renumbered REF** to mount
Changed lines of the file:
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@@
     (tags "mounting hole 4mm no annular")
     (attr exclude_from_pos_files exclude_from_bom)
-    (fp_text reference "REF**" (at 0 -5) (layer "F.SilkS")
+    (fp_text reference "mount" (at 0 -5) (layer "F.SilkS")
       (effects (font (size 1 1) (thickness 0.15)))
     )

Commit message: updated to latest design
Parts:
- removed J4: UART, Connector_PinHeader_2.54mm:PinHeader_1x04_P2.54mm_Vertical
- removed RST: RST, Button_Switch_SMD:SW_SPST_CK_RS282G05A3
- removed SW3: Set H, Button_Switch_SMD:SW_SPST_CK_RS282G05A3
- removed mount: MountingHole_4mm, MountingHole:MountingHole_4mm
- added H1: MountingHole, MountingHole:MountingHole_3.2mm_M3, F.Cu at (193.0, 102.5)
- added H2: MountingHole, MountingHole:MountingHole_3.2mm_M3, F.Cu at (160.0, 125.0)
- added H3: MountingHole, MountingHole:MountingHole_3.2mm_M3, F.Cu at (127.0, 102.5)
- added J2: UART, Connector_PinHeader_2.54mm:PinHeader_1x04_P2.54mm_Vertical, F.Cu at (103.0, 84.7)
- added RST1: RES, Button_Switch_SMD:SW_SPST_CK_RS282G05A3, F.Cu at (144.5, 88.0)
- added SW1: Set M, Button_Switch_SMD:SW_SPST_CK_RS282G05A3, F.Cu at (203.0, 88.1)
- D1: footprint LED_THT:LED_D5.0mm -> LED_SMD:LED_1206_3216Metric
- D3: footprint LED_SMD:LED_1206_3216Metric -> LED_THT:LED_D5.0mm
- R1, R2, R3: footprint Resistor_SMD:R_1206_3216Metric_Pad1.30x1.75mm_HandSolder -> Resistor_SMD:R_0805_2012Metric_Pad1.20x1.40mm_HandSolder
- SW2: value Set M -> Set H
- moved R2 36.8 mm to (193.5, 88.1)
- moved D3 24.0 mm to (163.0, 89.4)
- moved R3 10.0 mm to (172.0, 88.1)
- moved D4 5.50 mm to (168.5, 88.1)
- moved D2 4.00 mm to (184.5, 89.4)
- moved D1 3.73 mm to (190.0, 88.1)
- moved C1 2.79 mm to (169.0, 110.0)
- moved C2 2.79 mm to (169.0, 103.0)
- moved Y1 2.79 mm to (170.2, 105.5)
- moved U5 2.22 mm to (157.5, 106.5)
- moved SW2 1.00 mm to (213.0, 88.1)
- moved NU2 0.77 mm to (139.1, 104.8)
- moved NU3 0.49 mm to (181.5, 104.8)
- moved R1 0.10 mm to (151.5, 88.1)
Connections:
- net RST renamed RES
- D1 pad 2: Net-(D1-Pad2) -> Net-(D2-Pad2)
- D3 pad 2: Net-(D1-Pad2) -> Net-(D3-Pad2)
- D4 pad 2: Net-(D2-Pad2) -> Net-(D3-Pad2)
- R2 pad 2: Net-(D1-Pad2) -> Net-(D2-Pad2)
- R3 pad 2: Net-(D2-Pad2) -> Net-(D3-Pad2)
- SW2 pad 1: Net-(SW2-Pad1) -> SETH
- U1 pad 3: SD3 -> SD1
- U1 pad 9: G3 -> G1
- U2 pad 3: SD1 -> SD2
- U2 pad 9: G1 -> G2
- U3 pad 3: SD2 -> SD3
- U3 pad 9: G2 -> G3
- U5 pad 12: D1 -> SETM
- U5 pad 13: Net-(SW2-Pad1) -> D1
- U5 pad 14: Net-(SW3-Pad1) -> D2
- U5 pad 19: unconnected-(U5-Pad19) -> GNDREF
- U5 pad 22: unconnected-(U5-Pad22) -> GNDREF
- U5 pad 26: D2 -> SETH
Routing:
- net Net-(SW2-Pad1): track 75.8 -> 0.00 mm
- net SETH: track 0.00 -> 72.7 mm, vias 0 -> 2
- net Net-(SW3-Pad1): track 64.7 -> 0.00 mm
- net SETM: track 0.00 -> 47.1 mm
- net Net-(D1-Pad2): track 38.1 -> 0.00 mm
- net SD3: track 58.7 -> 26.2 mm, vias 2 -> 0
- net G3: track 69.8 -> 40.3 mm, vias 2 -> 0
- net D1: track 14.5 -> 39.1 mm
- net SD1: track 30.7 -> 54.5 mm, vias 0 -> 2
- net GNDREF: track 411.8 -> 433.2 mm, vias 2 -> 1
- net VCC: track 302.8 -> 282.5 mm, vias 2 -> 3
- net G1: track 25.6 -> 44.0 mm, vias 0 -> 2
- net G4: track 63.4 -> 81.7 mm
- net RXD: track 78.8 -> 62.6 mm, vias 1 -> 0
- net G2: track 37.5 -> 23.0 mm
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