File: hw/numitron clock.kicad_sch (KiCad schematic)
At the start: 24 parts, among them J1 AVR-ISP-6, J2 rtc, J3 5v in, J4 UART, SW1 RST, SW2 Set M, SW3 Set H, U1 TPIC6595, U2 TPIC6595, U3 TPIC6595, U4 TPIC6595, U5 ATmega8L-8A, Y1 Crystal

Commit message: version of pcb with more smd components
Parts:
- removed J2: rtc, Connector_PinHeader_2.54mm:PinHeader_1x05_P2.54mm_Vertical, symbol Connector:Conn_01x05_Male
- added D3, D4: LED, LED_SMD:LED_1206_3216Metric, symbol Device:LED
- R1, R2, R3: footprint Resistor_THT:R_Axial_DIN0207_L6.3mm_D2.5mm_P7.62mm_Horizontal -> Resistor_SMD:R_1206_3216Metric_Pad1.30x1.75mm_HandSolder
- U1, U2, U3, U4: footprint Package_DIP:DIP-20_W7.62mm_LongPads -> Package_SO:SOIC-20W_7.5x12.8mm_P1.27mm
- renumbered SW1 to RST
Connections:
- net G1: now also U5.28 (PC5); no longer J4.2 (Pin_2), U5.31 (PD1)
- net GNDREF: now also D3.1 (K), D4.1 (K)
- net SD1: now also U5.27 (PC4); no longer J4.3 (Pin_3), U5.30 (PD0)
- net at NU2.2 (DP): now also U2.4 (DRAIN0); no longer U2.7 (DRAIN3)
- net at NU2.3 (B): now also U2.5 (DRAIN1); no longer U2.6 (DRAIN2)
- net at NU2.4 (C): now also U2.6 (DRAIN2); no longer U2.5 (DRAIN1)
- net at NU2.5 (A): now also U2.7 (DRAIN3); no longer U2.4 (DRAIN0)
- net at NU2.6 (F): now also U2.15 (DRAIN5); no longer U2.14 (DRAIN4)
- net at NU2.7 (G): now also U2.16 (DRAIN6); no longer U2.17 (DRAIN7)
- net at NU2.8 (D): now also U2.17 (DRAIN7); no longer U2.16 (DRAIN6)
- net at NU2.9 (E): now also U2.14 (DRAIN4); no longer U2.15 (DRAIN5)
- net at NU4.2 (DP): now also U4.4 (DRAIN0); no longer U4.7 (DRAIN3)
- net at NU4.3 (B): now also U4.5 (DRAIN1); no longer U4.6 (DRAIN2)
- net at NU4.4 (C): now also U4.6 (DRAIN2); no longer U4.5 (DRAIN1)
- net at NU4.5 (A): now also U4.7 (DRAIN3); no longer U4.4 (DRAIN0)
- net at NU4.6 (F): now also U4.15 (DRAIN5); no longer U4.14 (DRAIN4)
- net at NU4.7 (G): now also U4.16 (DRAIN6); no longer U4.15 (DRAIN5)
- net at NU4.8 (D): now also U4.17 (DRAIN7); no longer U4.16 (DRAIN6)
- net at NU4.9 (E): now also U4.14 (DRAIN4); no longer U4.17 (DRAIN7)
- net at NU3.2 (DP): now also U3.4 (DRAIN0); no longer U3.7 (DRAIN3)
- net at NU3.3 (B): now also U3.5 (DRAIN1); no longer U3.6 (DRAIN2)
- net at NU3.4 (C): now also U3.6 (DRAIN2); no longer U3.5 (DRAIN1)
- net at NU3.5 (A): now also U3.7 (DRAIN3); no longer U3.4 (DRAIN0)
- net at NU3.6 (F): now also U3.15 (DRAIN5); no longer U3.14 (DRAIN4)
- net at NU3.7 (G): now also U3.16 (DRAIN6); no longer U3.17 (DRAIN7)
- net at NU3.8 (D): now also U3.17 (DRAIN7); no longer U3.16 (DRAIN6)
- net at NU3.9 (E): now also U3.14 (DRAIN4); no longer U3.15 (DRAIN5)
- net at NU1.2 (DP): now also U1.4 (DRAIN0); no longer U1.7 (DRAIN3)
- net at NU1.3 (B): now also U1.5 (DRAIN1); no longer U1.6 (DRAIN2)
- net at NU1.4 (C): now also U1.6 (DRAIN2); no longer U1.5 (DRAIN1)
- net at NU1.5 (A): now also U1.7 (DRAIN3); no longer U1.4 (DRAIN0)
- net at NU1.6 (F): now also U1.15 (DRAIN5); no longer U1.14 (DRAIN4)
- net at NU1.7 (G): now also U1.16 (DRAIN6); no longer U1.15 (DRAIN5)
- net at NU1.8 (D): now also U1.17 (DRAIN7); no longer U1.16 (DRAIN6)
- net at NU1.9 (E): now also U1.14 (DRAIN4); no longer U1.17 (DRAIN7)
- net at D1.2 (A), R2.2: now also D3.2 (A)
- net at D2.2 (A), R3.2: now also D4.2 (A)
- new net RXD: J4.2 (Pin_2), U5.30 (PD0)
- new net TXD: J4.3 (Pin_3), U5.31 (PD1)
Other:
- moved on the sheet: NU1, NU2, NU3, NU4

Commit message: updated to latest design
Parts:
- added H1, H2, H3: MountingHole, MountingHole:MountingHole_3.2mm_M3, symbol Mechanical:MountingHole
- R1, R2, R3: footprint Resistor_SMD:R_1206_3216Metric_Pad1.30x1.75mm_HandSolder -> Resistor_SMD:R_0805_2012Metric_Pad1.20x1.40mm_HandSolder
- RST1: renamed from RST; value RST -> RES
- renumbered D3 to D1, D1 to D2, D2 to D3, J4 to J2, NU2 to NU1, NU3 to NU2, NU1 to NU3, SW2 to SW1, SW3 to SW2, U2 to U1, U3 to U2, U1 to U3
Connections:
- net D1: now also U5.13 (PB1); no longer U5.12 (PB0)
- net D2: now also U5.14 (PB2); no longer U5.26 (PC3)
- net GNDREF: now also U5.19 (ADC6), U5.22 (ADC7)
- net SETM: now reaches SW1.1
- net SETM: now also U5.12 (PB0); no longer U5.13 (PB1)
- net SETH: now reaches SW2.1
- net SETH: now also U5.26 (PC3); no longer U5.14 (PB2)
- net RST renamed RES
Other:
- moved on the sheet: SW1, SW2

Commit message: final release?
Parts:
- added NU?: Numitron_IV-9, Numitron:numitron iv-9, symbol numitron:Numitron_IV-9-Display
- R1: value R -> 6k
- R2, R3: value R -> 130
Changed lines of the file:
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@@
       (effects (font (size 1.27 1.27)) (justify left))
     )
-    (property "Value" "R" (id 1) (at 61.468 23.4566 0)
+    (property "Value" "6k" (id 1) (at 61.468 23.4566 0)
       (effects (font (size 1.27 1.27)) (justify left))
     )
@@
     (in_bom yes) (on_board yes)
     (property "Reference" "R2" (id 0) (at 143.51 17.78 90))
-    (property "Value" "R" (id 1) (at 143.51 15.5726 90))
+    (property "Value" "130" (id 1) (at 143.51 15.5726 90))
     (property "Footprint" "Resistor_SMD:R_0805_2012Metric_Pad1.20x1.40mm_HandSolder" (id 2) (at 143.51 19.558 90)
       (effects (font (size 1.27 1.27)) hide)
@@
     (pin "1")
   )
+  (symbol (lib_id "numitron:Numitron_IV-9-Display") (at 189.23 152.4 0) (unit 1)
+    (in_bom yes) (on_board yes)
+    (property "Reference" "NU?" (id 0) (at 189.23 159.3342 0))
+    (property "Value" "Numitron_IV-9" (id 1) (at 189.23 161.6456 0))
+    (property "Footprint" "Numitron:numitron iv-9" (id 2) (at 189.23 167.64 0)
+      (effects (font (size 1.27 1.27)) hide)
+    )
+    (property "Datasheet" "http://www.kingbright.com/attachments/file/psearch/000/00/00/KCSA02-105(Ver.10A).pdf" (id 3) (at 176.53 140.335 0)
+      (effects (font (size 1.27 1.27)) (justify left) hide)
+    )
+    (pin "1")
+    (pin "2")
+    (pin "3")
+    (pin "4")
+    (pin "5")
+    (pin "6")
+    (pin "7")
+    (pin "8")
+    (pin "9")
+  )
   (symbol (lib_id "power:PWR_FLAG") (at 130.81 31.75 0) (unit 1)
     (in_bom yes) (on_board yes)
@@
     (in_bom yes) (on_board yes)
     (property "Reference" "R3" (id 0) (at 143.51 21.59 90))
-    (property "Value" "R" (id 1) (at 143.51 19.3826 90))
+    (property "Value" "130" (id 1) (at 143.51 19.3826 90))
     (property "Footprint" "Resistor_SMD:R_0805_2012Metric_Pad1.20x1.40mm_HandSolder" (id 2) (at 143.51 23.368 90)
       (effects (font (size 1.27 1.27)) hide)
@@
       (reference "NU4") (unit 1) (value "Numitron_IV-9") (footprint "Numitron:numitron iv-9")
     )
+    (path "/ed01385c-df22-4d74-a0f1-02529dbaa5bf"
+      (reference "NU?") (unit 1) (value "Numitron_IV-9") (footprint "Numitron:numitron iv-9")
+    )
     (path "/30f6ac74-f501-4148-81d0-578662cc8067"
-      (reference "R1") (unit 1) (value "R") (footprint "Resistor_SMD:R_0805_2012Metric_Pad1.20x1.40mm_HandSolder")
+      (reference "R1") (unit 1) (value "6k") (footprint "Resistor_SMD:R_0805_2012Metric_Pad1.20x1.40mm_HandSolder")
     )
     (path "/b8c29b55-b764-44a2-8453-ce2092d7b392"
-      (reference "R2") (unit 1) (value "R") (footprint "Resistor_SMD:R_0805_2012Metric_Pad1.20x1.40mm_HandSolder")
+      (reference "R2") (unit 1) (value "130") (footprint "Resistor_SMD:R_0805_2012Metric_Pad1.20x1.40mm_HandSolder")
     )
     (path "/f9826504-d549-46c5-b2e9-d7a87f63fc59"
-      (reference "R3") (unit 1) (value "R") (footprint "Resistor_SMD:R_0805_2012Metric_Pad1.20x1.40mm_HandSolder")
+      (reference "R3") (unit 1) (value "130") (footprint "Resistor_SMD:R_0805_2012Metric_Pad1.20x1.40mm_HandSolder")
     )
     (path "/bfa58ffe-75b4-4ffe-b7ce-22611df5a49a"
